File: KiCad/SaturnGeoCar/SaturnGeoCar.kicad_sch (KiCad schematic)
At the start: 3 parts, among them J1 1054500101, U1 ESP32-WROVER-E-N16R8, U2 MCP1700-3302E_TO

Commit message: Finished uploading all components, wiring has started
Parts:
- added BT1, BT2: XT60-F, Connector_AMASS:AMASS_XT60-F_1x02_P7.20mm_Vertical, symbol Device:Battery_Cell
- added C1, C5: 22uF 12V, symbol Device:C
- added C2, C6: 220pF 12V, symbol Device:C
- added C3, C7: 100nf, symbol Device:C
- added C4, C8: 10uF, symbol Device:C
- added C9: 22uF, symbol Device:C
- added D1, D2: 20V 3A, symbol Device:D
- added D3, D4: SS34, symbol Device:D
- added IC1: SHT30-ARP-B2.5KS, SHT30-ARP-B2.5KS:SON50P250X250X100-9N-D, symbol SHT30-ARP-B2_5KS:SHT30-ARP-B2.5KS
- added IC2: TSL25911FN, TSL25911FN:TSL25911FN, symbol TSL25911FN:TSL25911FN
- added IC3: SN74HC165NSR, SN74HC165NSR:SOIC127P780X200-16N, symbol SN74HC165NSR:SN74HC165NSR
- added IC4, IC5, IC6, IC7: DRV8300DPWR, DRV8300DPWR:SOP65P640X120-20N, symbol DRV8300DPWR:DRV8300DPWR
- added J2, J3: U.FL-R-SMT-1_80_, U.FL-R-SMT-1_80_:HIROSE_U.FL-R-SMT-1_80_, symbol U.FL-R-SMT-1_80_:U.FL-R-SMT-1_80_
- added J4: FFC2B28-24-G, FFC2B28-24-G:GCT_FFC2B28-24-G, symbol FFC2B28-24-G:FFC2B28-24-G
- added J5, J6, J7, J8: WJ126V-5.0-3P, WJ126V-5.0-3P:WJ126V503P, symbol WJ126V-5_0-3P:WJ126V-5.0-3P
- added L1, L2: 10 uH 3A <35 mOhm, symbol Device:L
- added MICRO_SD1: TF-01A, TF-01A:TF-01A, symbol TF-01A:TF-01A
- added MK1: SPH0641LU4H-1, SPH0641LU4H-1:MIC_SPH0641LU4H-1, symbol SPH0641LU4H-1:SPH0641LU4H-1
- added R1, R6: 127k 1%, symbol Device:R
- added R10, R5: 180k, symbol Device:R
- added R2: 40.2K 1%, symbol Device:R
- added R3, R8: 68.1k 1%, symbol Device:R
- added R4, R9: 1k, symbol Device:R
- added R7: 31.6kK 1%, symbol Device:R
- added S1, S2, S3: KMR221GLFS, KMR221GLFS:KMR231GLFS, symbol KMR221GLFS:KMR221GLFS
- added U10: BMP388, BMP388:PQFN50P200X200X80-10N, symbol BMP388:BMP388
- added U11: SIM7600G, SIM7600G:IC_SIM7600G, symbol SIM7600G:SIM7600G
- added U12, U6: MP1584EN-LF-Z, MP1584EN-LF-Z:SOIC127P600X170-9N, symbol MP1584EN-LF-Z:MP1584EN-LF-Z
- added U3: LSM6DS3TR-C, LSM6DS3TR-C:LGA-14-2.5X3MM, symbol LSM6DS3TR-C:LSM6DS3TR-C
- added U4: LIS3MDLTR, LIS3MDLTR:XDCR_LIS3MDLTR, symbol LIS3MDLTR:LIS3MDLTR
- added U5: MAX17048G_T10, MAX17048G_T10:SON50P200X200X80-9N, symbol MAX17048G_T10:MAX17048G_T10
- added U7: MAX98357AETE_T, MAX98357AETE_T:QFN50P300X300X80-17N, symbol MAX98357AETE_T:MAX98357AETE_T
- added U8: PCF8563T_5_518, PCF8563T_5_518:SOIC127P599X175-8N, symbol PCF8563T_5_518:PCF8563T_5_518
- added U9: CR2032-BS-5-1, CR2032-BS-5-1:CR2032BS51, symbol CR2032-BS-5-1:CR2032-BS-5-1
Connections:
- net GND: now also U2.1 (GND), BT1.2 (-), BT2.2 (-), C1.1, C4.2, C5.1, C8.2, D1.2 (A), D2.2 (A), IC2.3 (GND), J2.G1, J2.G2, J3.G1, J3.G2, J4.S1 (SHIELD), J4.S2 (SHIELD), MICRO_SD1.MP1 (SHIELD), MICRO_SD1.MP2 (SHIELD), MICRO_SD1.MP3 (SHIELD), MICRO_SD1.MP4 (SHIELD), MK1.3 (GND), R10.1, R2.2, R3.1, R4.1, R5.1, R7.2, R8.1, R9.1, U12.5 (GND), U12.9 (EP), U3.6 (GND), U3.7 (GND), U4.3 (GND), U5.4 (GND), U6.5 (GND), U6.9 (EP), U7.11 (GND), U7.15 (GND), U7.3 (GND)
- net +5V: now reaches U2.2 (VIN)
- net at U2.3 (VOUT): now also D3.2 (A)
- new net: R5.2, U6.6 (FREQ)
- new net: R6.2, R7.1, U12.4 (FB)
- new net: C6.1, R8.2
- new net: C1.2, D4.2 (A), L1.2, R1.1
- new net: R1.2, R2.1, U6.4 (FB)
- new net: C9.2, D3.1 (K), D4.1 (K)
- new net: C3.1, D1.1 (K), L1.1, U6.1 (SW)
- new net: C3.2, U6.8 (BST)
- new net: U11.1 (GND), U11.10 (GND), U11.110 (GND), U11.118 (GND), U11.120 (GND), U11.121 (GND), U11.122 (GND), U11.123 (GND), U11.124 (GND), U11.125 (GND), U11.126 (GND), U11.127 (GND), U11.128 (GND), U11.129 (GND), U11.130 (GND), U11.131 (GND), U11.132 (GND), U11.133 (GND), U11.134 (GND), U11.135 (GND), U11.14 (GND), U11.2 (GND), U11.37 (GND), U11.40 (GND), U11.41 (GND), U11.43 (GND), U11.5 (GND), U11.57 (GND), U11.58 (GND), U11.60 (GND), U11.61 (GND), U11.64 (GND), U11.65 (GND), U11.77 (GND), U11.78 (GND), U11.80 (GND), U11.81 (GND), U11.93 (GND), U11.98 (GND)
- new net: U11.38 (VBAT), U11.39 (VBAT), U11.62 (VBAT), U11.63 (VBAT)
- new net: R4.2, U6.2 (EN)
- new net: C2.2, U6.3 (COMP)
- new net: C7.1, D2.1 (K), L2.1, U12.1 (SW)
- new net: U11.100 (RESERVED), U11.101 (RESERVED), U11.102 (RESERVED), U11.103 (RESERVED), U11.104 (RESERVED), U11.105 (RESERVED), U11.111 (RESERVED), U11.88 (RESERVED), U11.89 (RESERVED), U11.90 (RESERVED), U11.91 (RESERVED), U11.92 (RESERVED), U11.99 (RESERVED)
- new net: U10.3 (VSS), U10.8 (VSS), U10.9 (VSS)
- new net: C2.1, R3.2
- new net: R10.2, U12.6 (FREQ)
- new net: C6.2, U12.3 (COMP)
- new net: C7.2, U12.8 (BST)
- new net: R9.2, U12.2 (EN)
- new net: U7.7 (VDD), U7.8 (VDD)
- new net +11.1V: BT1.1 (+), BT2.1 (+), C4.1, C8.1, U12.7 (VIN), U6.7 (VIN)
- new net +3V3: C9.1
- new net +4V: C5.2, L2.2, R6.1
Other:
- note added: "11.1V to 3V3"
- note added: "11.1V to 4V"
- note added: "3D Magnetic Sensor"
- note added: "BLDC driver + Motor connectors"
- note added: "Barometric sensor"
- note added: "Battery"
- note added: "Battery Connectors"
- note added: "Boot"
- note added: "Buttons"
- note added: "Camera"
- note added: "Coin Cell DO NOT POWER ANYTHING FROM THIS"
- note added: "Extra"
- note added: "Fuel gauge IC"
- note added: "GPS + SIM"
- note added: "IMU"
- note added: "Light + UV sensor"
- note added: "Micro SD"
- note added: "Microphone"
- note added: "Parallel-in shift reg."
- note added: "RTC IC"
- note added: "Reset"
- note added: "SENSORS"
- note added: "Speaker Amp"
- note added: "Temp + Humidity sensor"
- moved on the sheet: J1, U2

Commit message: updated a few parts
Parts:
- added D?: TPD2E001DZDR, TPD2E001DZDR, symbol TPD2E001DZDR:TPD2E001DZDR
- added R11, R12: 5.1k, symbol Device:R
Connections:
- net +5V: now also J1.A4 (VBUS_A4), J1.A9 (VBUS_A9), J1.B4 (VBUS_B4), J1.B9 (VBUS_B9)
- net GND: now also J1.SH1 (SHIELD3), J1.SH2 (SHIELD4), J1.SH3 (SHIELD1), J1.SH4 (SHIELD2), D?.1 (GND), R11.1, R12.2
- net at J1.A5 (CC1): now also R11.2
- net D+: now reaches J1.A6 (D1+)
- net D+: now also J1.B6 (D2+), D?.2 (IO1)
- net D-: now reaches J1.A7 (D1-)
- net D-: now also J1.B7 (D2-), D?.3 (IO2)
- net at J1.B5 (CC2): now also R12.1
- no-connect marks 0 -> 12
Other:
- moved on the sheet: C9, D3, D4, J1, U2

Commit message: finshed adding all componets, everything is wired properly. Adding solar panel next
Parts:
- removed IC1: SHT30-ARP-B2.5KS, SHT30-ARP-B2.5KS:SON50P250X250X100-9N-D, symbol SHT30-ARP-B2_5KS:SHT30-ARP-B2.5KS
- removed IC3: SN74HC165NSR, SN74HC165NSR:SOIC127P780X200-16N, symbol SN74HC165NSR:SN74HC165NSR
- removed IC4, IC5, IC6, IC7: DRV8300DPWR, DRV8300DPWR:SOP65P640X120-20N, symbol DRV8300DPWR:DRV8300DPWR
- removed S3: KMR221GLFS, KMR221GLFS:KMR231GLFS, symbol KMR221GLFS:KMR221GLFS
- removed U1: ESP32-WROVER-E-N16R8, footprints:ESP32-WROVER-E_EXP, symbol Espressif:ESP32-WROVER-E-N16R8
- removed U2: MCP1700-3302E_TO, MCP1700-3302E_TO:TO127P254X495-3, symbol MCP1700-3302E_TO:MCP1700-3302E_TO
- removed U5: MAX17048G_T10, MAX17048G_T10:SON50P200X200X80-9N, symbol MAX17048G_T10:MAX17048G_T10
- removed U8: PCF8563T_5_518, PCF8563T_5_518:SOIC127P599X175-8N, symbol PCF8563T_5_518:PCF8563T_5_518
- added C10, C11, C29, C30, C32, C35, C36, C38, C41, C42, C44, C47, C48, C50, C53, C55: 1uF, symbol Device:C
- added C12, C15, C16, C17, C18, C19, C21, C22, C24, C25, C26, C27, C31, C33, C37, C39, C43, C45, C49, C51: 0.1uF, symbol Device:C
- added C13, C14: 100nF, symbol Device:C
- added C20, C28, C34, C40, C46: 10uF, symbol Device:C
- added C23: 4.7uF, symbol Device:C
- added C52: 1000µF, symbol Device:C
- added C54: 1µF, symbol Device:C
- added C56: 100Nf, symbol Device:C
- added C57, C58: 20pF, symbol Device:C
- added D10, D6, D7, D8, D9: LED, symbol Device:LED
- added IC1: SHT31-DIS-B2.5KS, SHT31-DIS-B2.5KS:SON50P250X250X100-9N-D, symbol SHT31-DIS-B2_5KS:SHT31-DIS-B2.5KS
- added IC3: MCP23017-E_SO, MCP23017-E_SO:SOIC127P1030X265-28N, symbol MCP23017-E_SO:MCP23017-E_SO
- added IC4, IC5, IC6, IC8: DRV10983PWPR, DRV10983PWPR:SOP65P640X120-25N, symbol DRV10983PWPR:DRV10983PWPR
- added IC7: AP2112K-1.8TRG1, AP2112K-1.8TRG1:SOT95P285X140-5N, symbol AP2112K-1_8TRG1:AP2112K-1.8TRG1
- added J10: SIM8055-6-1-14-01-A, SIM8055-6-1-14-01-A:SIM8055611401A, symbol SIM8055-6-1-14-01-A:SIM8055-6-1-14-01-A
- added J9: WJ126V-5.0-2P, WJ126V-5.0-2P:SHDR2W105P0X500_1X2_1000X780X1040P, symbol WJ126V-5_0-2P:WJ126V-5.0-2P
- added L3, L4, L5, L6: 47uH, symbol Device:L
- added R13, R14, R18: 100k, symbol Device:R
- added R15, R16, R19, R21, R22, R23, R24, R25, R26: 10k, symbol Device:R
- added R17: 0.1, symbol Device:R
- added R20: 1k, symbol Device:R
- added R27: 3.7k, symbol Device:R
- added R28: 100, symbol Device:R
- added U1: ESP32-S3, ESP32-S3:IC_ESP32-S3, symbol ESP32-S3:ESP32-S3
- added U13: W25Q128JVSIQ, W25Q128JVSIQ:SOIC127P790X216-8N, symbol W25Q128JVSIQ:W25Q128JVSIQ
- added U14: CH340C, CH340C:SOIC127P600X180-16N, symbol CH340C:CH340C
- added U15: BME680, BME680:PSON80P300X300X100-8N, symbol BME680:BME680
- added U2: AP2112K-3.3TRG1, AP2112K-3.3TRG1:SOT95P285X140-5N, symbol AP2112K-3.3TRG1:AP2112K-3.3TRG1
- added U5: INA219AID, INA219AID:SOIC127P599X175-8N, symbol INA219AID:INA219AID
- added U8: DS3231SN_T_R, DS3231SN_T_R:SOIC127P1032X265-16N, symbol DS3231SN_T_R:DS3231SN_T_R
- added X1: X321532768KGD2SI, PCM_JLCPCB:CRYSTAL-SMD_L11.5-W4.8-LS12.7, symbol PCM_JLCPCB-Crystals:Crystal, 8MHz, 20pF, ±20ppm
- added Y1: X322540MPB4SI, X322540MPB4SI:X322540MPB4SI, symbol X322540MPB4SI:X322540MPB4SI
- D5: renamed from D?; footprint TPD2E001DZDR -> TPD2E001DZDR:TPD2E001DZDR
Connections:
- net +11.1V: now also C33.2, C39.2, C45.2, C51.2, IC4.23 (VCC_1), IC4.24 (VCC_2), IC5.23 (VCC_1), IC5.24 (VCC_2), IC6.23 (VCC_1), IC6.24 (VCC_2), IC8.23 (VCC_1), IC8.24 (VCC_2), R17.2, U5.7 (VIN-)
- net +3V3: now also IC2.5 (VDD), J4.1, J4.2, J4.3, MICRO_SD1.4 (VDD), MK1.5 (VDD), U10.1 (VDDIO), U10.10 (VDD), U10.6 (CSB), U3.12 (CS), U3.5 (VDDIO), U3.8 (VDD), U4.10 (CS), U4.5 (VDD), U4.6 (VDD_IO), U7.7 (VDD), U7.8 (VDD), C12.1, C15.1, C16.1, C18.1, C19.1, C20.1, C21.1, C22.2, C24.1, C25.1, C26.1, C27.1, IC1.5 (VDD), IC1.6 (NRESET), IC3.9 (VDD), R13.1, R14.1, R15.1, R16.2, R18.1, R19.2, R21.2, R26.1, U1.2 (VDD3P3), U1.20 (VDD3P3_RTC), U1.29 (VDD_SPI), U1.3 (VDD3P3), U1.46 (VDD3P3_CPU), U1.55 (VDDA1), U1.56 (VDDA2), U13.8 (VCC), U14.16 (VCC), U15.2 (CSB), U15.6 (VDDIO), U15.8 (VDD), U5.5 (VS), U8.2 (VCC)
- net +4V: now also C52.1, C54.1
- net +5V: now also U11.11 (USB_VBUS), C10.1, C53.1, IC7.1 (VIN), IC7.3 (EN), U2.1 (VIN), U2.3 (EN)
- net D+: now also U11.13 (USB_DP), U1.27 (GPIO21), U14.5 (UD+)
- net D-: now also U11.12 (USB_DN), U1.26 (GPIO20), U14.6 (UD-)
- net GND: now also J4.24, J4.4, J4.5, J4.8, MICRO_SD1.6 (VSS), MK1.2 (SELECT), S1.2 (NO_1), S1.5 (GND), S2.2 (NO_1), S2.5 (GND), U10.3 (VSS), U10.5 (SDO), U10.8 (VSS), U10.9 (VSS), U11.1 (GND), U11.10 (GND), U11.110 (GND), U11.118 (GND), U11.120 (GND), U11.121 (GND), U11.122 (GND), U11.123 (GND), U11.124 (GND), U11.125 (GND), U11.126 (GND), U11.127 (GND), U11.128 (GND), U11.129 (GND), U11.130 (GND), U11.131 (GND), U11.132 (GND), U11.133 (GND), U11.134 (GND), U11.135 (GND), U11.14 (GND), U11.2 (GND), U11.37 (GND), U11.40 (GND), U11.41 (GND), U11.43 (GND), U11.5 (GND), U11.57 (GND), U11.58 (GND), U11.60 (GND), U11.61 (GND), U11.64 (GND), U11.65 (GND), U11.77 (GND), U11.78 (GND), U11.80 (GND), U11.81 (GND), U11.83 (COEX1), U11.84 (COEX2), U11.86 (COEX3), U11.93 (GND), U11.98 (GND), U3.1 (SDO/SA0), U4.12 (RSVD2), U4.2 (RSVD1), U4.9 (SDO/SA1), U7.17 (EP), U7.2 (GAIN_SLOT), U7.4 (SD_MODE), U9.3 (-), C10.2, C11.2, C12.2, C15.2, C16.2, C17.2, C18.2, C19.2, C20.2, C21.2, C22.1, C23.2, C24.2, C25.2, C26.2, C27.2, C28.1, C29.1, C30.1, C32.1, C34.1, C35.1, C36.1, C38.1, C40.1, C41.1, C42.1, C44.1, C46.1, C47.1, C48.1, C50.1, C53.2, C54.2, C55.2, C56.1, C57.1, C58.1, D10.1 (K), D6.1 (K), D7.1 (K), D8.1 (K), D9.1 (K), IC1.2 (ADDR), IC1.8 (VSS), IC1.9 (EP), IC3.10 (VSS), IC3.15 (A0), IC3.16 (A1), IC3.17 (A2), IC4.15 (PGND_1), IC4.16 (PGND_2), IC4.25 (THERMAL_PAD_(GND)), IC4.5 (SWGND), IC4.8 (GND), IC5.15 (PGND_1), IC5.16 (PGND_2), IC5.25 (THERMAL_PAD_(GND)), IC5.5 (SWGND), IC5.8 (GND), IC6.15 (PGND_1), IC6.16 (PGND_2), IC6.25 (THERMAL_PAD_(GND)), IC6.5 (SWGND), IC6.8 (GND), IC7.2 (GND), IC8.15 (PGND_1), IC8.16 (PGND_2), IC8.25 (THERMAL_PAD_(GND)), IC8.5 (SWGND), IC8.8 (GND), J10.C5 (GND), J10.MH1, J10.MH2, J10.MP1, J10.MP2, R17.1, R22.1, R23.1, R24.1, R25.1, U1.57 (GND), U13.4 (GND), U14.1 (GND), U15.1 (GND), U15.5 (SDO), U15.7 (GND), U2.2 (GND), U5.1 (A1), U5.2 (A0), U5.6 (GND), U5.8 (VIN+), U8.13 (GND), Y1.2 (GND_1), Y1.4 (GND_2)
- net SDDAT3: now reaches MICRO_SD1.2 (CD/DAT3)
- net SDDAT3: now also R25.2, U1.25 (GPIO19)
- net SDCMD: now reaches MICRO_SD1.3 (CMD)
- net SDCMD: now also R22.2, U1.19 (GPIO14)
- net SDCLK: now reaches MICRO_SD1.5 (CLK)
- net SDCLK: now also R24.2, U1.24 (GPIO18)
- net SDDAT0: now reaches MICRO_SD1.7 (DAT0)
- net SDDAT0: now also R23.2, U1.23 (GPIO17)
- net CardDetect: now reaches MICRO_SD1.CD1 (CD)
- net CardDetect: now also IC3.5 (GPB4)
- net SCL: now reaches U3.13 (SCL)
- net SCL: now also IC2.1 (SCL), J4.7, U10.2 (SCK), U11.55 (SCL), U4.1 (SCL/SPC), IC1.4 (SCL), IC3.12 (SCL), IC4.10 (SCL), IC5.10 (SCL), IC6.10 (SCL), IC8.10 (SCL), R15.2, U1.9 (GPIO4), U15.4 (SCK), U5.4 (SCL), U8.16 (SCL)
- net SDA: now reaches U3.14 (SDA)
- net SDA: now also IC2.6 (SDA), J4.6, U10.4 (SDI), U11.56 (SDA), U4.11 (SDA/SDI/SDO), IC1.1 (SDA), IC3.13 (SDA), IC4.11 (SDA), IC5.11 (SDA), IC6.11 (SDA), IC8.11 (SDA), R16.1, U1.10 (GPIO5), U15.3 (SDI), U5.3 (SDA), U8.15 (SDA)
- net GNSSA: now reaches J3.SIG
- net GNSSA: now also U11.79 (GNSS_ANT)
- net U3: now reaches J7.1
- net U3: now also IC6.17 (U_1), IC6.18 (U_2)
- net V3: now reaches J7.2
- net V3: now also IC6.19 (V_1), IC6.20 (V_2)
- net W3: now reaches J7.3
- net W3: now also IC6.21 (W_1), IC6.22 (W_2)
- net U2: now reaches J6.1
- net U2: now also IC5.17 (U_1), IC5.18 (U_2)
- net V2: now reaches J6.2
- net V2: now also IC5.19 (V_1), IC5.20 (V_2)
- net W2: now reaches J6.3
- net W2: now also IC5.21 (W_1), IC5.22 (W_2)
- net at D3.2 (A): now also C11.1, U2.5 (VOUT)
- net SIMDATA: now reaches U11.17 (USIM_DATA)
- net SIMDATA: now also J10.C7 (I/O)
- net SIMRESET: now reaches U11.18 (USIM_RST)
- net SIMRESET: now also J10.C2 (RST)
- net SIMCLK: now reaches U11.19 (USIM_CLK)
- net SIMCLK: now also J10.C3 (CLK)
- net SIMVCC: now reaches U11.20 (USIM_VDD)
- net SIMVCC: now also C56.2, J10.C1 (VCC)
- net PWRKEY: now reaches U11.3 (~{PWRKEY})
- net PWRKEY: now also R20.2, U1.14 (GPIO9)
- net at U11.38 (VBAT), U11.39 (VBAT), U11.62 (VBAT)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: now also C52.2
- net RESET: now reaches U11.4 (~{RESET})
- net RESET: now also J4.9, S1.1 (COM_1), C14.2, IC3.18 (~{RESET}), R21.1, R26.2, U1.4 (CHIP_PU), U1.43 (GPIO38)
- net NETLIGHT: now reaches U11.51 (NETLIGHT)
- net NETLIGHT: now also R28.2
- net SIMCD: now reaches U11.53 (USIM_DET)
- net SIMCD: now also J10.CD1 (CD)
- net at U11.54 (FLIGHTMODE): now also R27.2
- net uC_RX: now reaches U11.68 (RXD)
- net uC_RX: now also U1.50 (U0RXD), U1.7 (GPIO2), U14.3 (RXD)
- net uC_TX: now reaches U11.71 (TXD)
- net uC_TX: now also U1.49 (U0TXD), U1.6 (GPIO1), U14.2 (TXD)
- net LTEA: now reaches U11.82 (MAIN_ANT)
- net LTEA: now also J2.SIG
- net COM1: now reaches S2.1 (COM_1)
- net COM1: now also IC3.6 (GPB5)
- net at U9.1 (+_1): now also U9.2 (+_2), U8.14 (VBAT)
- net CAMXCLK: now reaches J4.10
- net CAMXCLK: now also J4.23, U1.44 (MTCK)
- net CAMPWDN: now reaches J4.11
- net CAMPWDN: now also U1.8 (GPIO3)
- net D0: now reaches J4.14
- net D0: now also U1.52 (GPIO46)
- net D1: now reaches J4.15
- net D1: now also U1.39 (GPIO34)
- net D2: now reaches J4.16
- net D2: now also U1.40 (GPIO35)
- net D3: now reaches J4.17
- net D3: now also U1.41 (GPIO36)
- net D4: now reaches J4.18
- net D4: now also U1.38 (GPIO33)
- net D5: now reaches J4.19
- net D5: now also U1.5 (GPIO0)
- net D6: now reaches J4.20
- net D6: now also U1.48 (MTMS)
- net D7: now reaches J4.21
- net D7: now also U1.47 (MTDI)
- net CAMPCLK: now reaches J4.22
- net CAMPCLK: now also U1.45 (MTDO)
- net at U4.4 (C1): now also C17.1
- net U4: now reaches J8.1
- net U4: now also IC8.17 (U_1), IC8.18 (U_2)
- net V4: now reaches J8.2
- net V4: now also IC8.19 (V_1), IC8.20 (V_2)
- net W4: now reaches J8.3
- net W4: now also IC8.21 (W_1), IC8.22 (W_2)
- net DATA: now reaches MK1.1 (DATA)
- net DATA: now also U1.51 (GPIO45)
- net BCLK: now reaches MK1.4 (CLOCK)
- net BCLK: now also U7.16 (BCLK), U1.11 (GPIO6)
- net U1: now reaches J5.1
- net U1: now also IC4.17 (U_1), IC4.18 (U_2)
- net V1: now reaches J5.2
- net V1: now also IC4.19 (V_1), IC4.20 (V_2)
- net W1: now reaches J5.3
- net W1: now also IC4.21 (W_1), IC4.22 (W_2)
- net DIN: now reaches U7.1 (DIN)
- net DIN: now also U1.13 (GPIO8)
- net NS: now reaches U7.10 (OUTN)
- net NS: now also J9.2
- net LRCLK: now reaches U7.14 (LRCLK)
- net LRCLK: now also U1.12 (GPIO7)
- net PS: now reaches U7.9 (OUTP)
- net PS: now also J9.1
- new net: IC5.4 (SW), L4.1
- new net: C34.2, L4.2
- new net: C57.2, U1.54 (XTAL_P), Y1.1 (CRYSTAL_1)
- new net: C44.2, IC6.6 (VREG)
- new net: C41.2, IC6.7 (V1P8)
- new net: C43.1, IC6.3 (CPN)
- new net: C43.2, IC6.2 (CPP)
- new net: C31.1, IC4.3 (CPN)
- new net: C31.2, IC4.2 (CPP)
- new net: C58.2, U1.53 (XTAL_N), Y1.3 (CRYSTAL_2)
- new net: C49.1, IC8.3 (CPN)
- new net: C49.2, IC8.2 (CPP)
- new net: C14.1, U14.13 (~{DTR})
- new net: IC4.4 (SW), L3.1
- new net: C28.2, L3.2
- new net: C13.1, U14.14 (~{RTS})
- new net: C23.1, U14.4 (V3)
- new net: C39.1, IC5.1 (VCP)
- new net: C37.2, IC5.2 (CPP)
- new net: C37.1, IC5.3 (CPN)
- new net: C38.2, IC5.6 (VREG)
- new net: C35.2, IC5.7 (V1P8)
- new net: C36.2, IC5.9 (V3P3)
- new net: D6.2 (A), R28.1
- new net: U1.21 (XTAL_32K_P), X1.1
- new net: U1.22 (XTAL_32K_N), X1.2
- new net: C33.1, IC4.1 (VCP)
- new net: C32.2, IC4.6 (VREG)
- new net: C29.2, IC4.7 (V1P8)
- new net: C30.2, IC4.9 (V3P3)
- new net: C45.1, IC6.1 (VCP)
- new net: C51.1, IC8.1 (VCP)
- new net: C48.2, IC8.9 (V3P3)
- new net: IC6.4 (SW), L5.1
- new net: C40.2, L5.2
- new net: C50.2, IC8.6 (VREG)
- new net: C42.2, IC6.9 (V3P3)
- new net: IC8.4 (SW), L6.1
- new net: C47.2, IC8.7 (V1P8)
- new net: C46.2, L6.2
- new net +1.8V: C55.1, IC7.5 (VOUT), R20.1, R27.1
- new net DIR1: IC3.1 (GPB0), IC4.14 (DIR)
- new net DIR2: IC3.2 (GPB1), IC5.14 (DIR)
- new net DIR3: IC3.3 (GPB2), IC6.14 (DIR)
- new net DIR4: IC3.4 (GPB3), IC8.14 (DIR)
- new net FCLK: U1.33 (SPICLK), U1.37 (SPICLK_P), U13.6 (CLK)
- new net FCS: R14.2, U1.32 (SPICS0), U13.1 (/CS)
- new net FIO0: U1.34 (SPIQ), U13.5 (DI(IO0))
- new net FIO1: U1.35 (SPID), U13.2 (DO(IO1))
- new net FIO2: R13.2, U1.31 (SPIWP), U13.3 (/WP(IO2))
- new net FIO3: R18.2, U1.30 (SPIHD), U13.7 (/HOLD/RESET(IO3))
- new net LED1: D10.2 (A), IC3.28 (GPA7)
- new net LED2: D9.2 (A), IC3.27 (GPA6)
- new net LED3: D8.2 (A), IC3.26 (GPA5)
- new net LED4: D7.2 (A), IC3.25 (GPA4)
- new net RESET_EN: C13.2, R19.1
- new net SPEED1: IC4.13 (SPEED), U1.18 (GPIO13)
- new net SPEED2: IC5.13 (SPEED), U1.17 (GPIO12)
- new net SPEED3: IC6.13 (SPEED), U1.16 (GPIO11)
- new net SPEED4: IC8.13 (SPEED), U1.15 (GPIO10)
- no-connect marks 12 -> 116
Other:
- note added: "5V to 1.8V"
- note added: "Air Quality/Gas Sensor"
- note added: "ESD prot."
- note added: "Free"
- note added: "GPIO Expander"
- note added: "LEDs"
- note added: "SPI Flash chip"
- note added: "Speaker"
- note added: "Speaker Connector"
- note added: "USB-to-Serial + BOOT"
- note removed: "Boot"
- note removed: "Parallel-in shift reg."
- moved on the sheet: BT1, BT2, C1, C2, C3, C4, D1, IC2, J2, J3, J4, J5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

Commit message: hehe easyeda sucks (almost done)
Connections:
- net D+: no longer U1.27 (GPIO21)
- net D-: no longer U1.26 (GPIO20)
- net FCLK: no longer U1.37 (SPICLK_P)
- net RESET: no longer U1.43 (GPIO38)
- no-connect marks 116 -> 120
Changed lines of the file:
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@@
 	)
 	(no_connect
+		(at 81.28 118.11)
+	)
+	(no_connect
 		(at 321.31 391.16)
 	)
@@
 	)
 	(no_connect
+		(at 30.48 100.33)
+	)
+	(no_connect
 		(at 175.26 214.63)
 	)
@@
 	)
 	(no_connect
+		(at 81.28 100.33)
+	)
+	(no_connect
 		(at 402.59 81.28)
 	)
 	(no_connect
+		(at 81.28 102.87)
+	)
+	(no_connect
 		(at 247.65 226.06)
 	)
@@
 	(wire
 		(pts
-			(xy 99.06 492.76) (xy 99.06 495.3)
-		)
-		(stroke
-			(width 0)
-			(type default)
-		)
-	)
-	(wire
-		(pts
 			(xy 308.61 492.76) (xy 308.61 495.3)
 		)
@@
 	(wire
 		(pts
+			(xy 99.06 492.76) (xy 99.06 495.3)
+		)
+		(stroke
+			(width 0)
+			(type default)
+		)
+	)
+	(wire
+		(pts
 			(xy 332.74 299.72) (xy 331.47 299.72)
 		)
@@
 		)
 	)
+	(text "Free"
+		(exclude_from_sim no)
+		(at 84.582 103.124 0)
+		(effects
+			(font
+				(size 1.27 1.27)
+			)
+		)
+	)
+	(text "Free"
+		(exclude_from_sim no)
+		(at 84.582 118.11 0)
+		(effects
+			(font
+				(size 1.27 1.27)
+			)
+		)
+	)
 	(text "Temp + Humidity sensor"
 		(exclude_from_sim no)
@@
 		)
 	)
+	(text "Free"
+		(exclude_from_sim no)
+		(at 84.582 100.584 0)
+		(effects
+			(font
+				(size 1.27 1.27)
+			)
+		)
+	)
 	(text "ESP-32"
 		(exclude_from_sim no)
@@
 		)
 	)
-	(global_label "D+"
-		(shape input)
-		(at 81.28 102.87 0)
-		(fields_autoplaced yes)
-		(effects
-			(font
-				(size 1.27 1.27)
-			)
-			(justify left)
-		)
-		(property "Intersheetrefs" "${INTERSHEET_REFS}"
-			(at 87.1076 102.87 0)
-			(effects
-				(font
-					(size 1.27 1.27)
-				)
-				(justify left)
-				(hide yes)
-			)
-		)
-	)
 	(global_label "LTEA"
 		(shape input)
@@
 		)
 	)
-	(global_label "FCLK"
-		(shape input)
-		(at 30.48 100.33 180)
-		(fields_autoplaced yes)
-		(effects
-			(font
-				(size 1.27 1.27)
-			)
-			(justify right)
-		)
-		(property "Intersheetrefs" "${INTERSHEET_REFS}"
-			(at 22.8381 100.33 0)
-			(effects
-				(font
-					(size 1.27 1.27)
-				)
-				(justify right)
-				(hide yes)
-			)
-		)
-	)
 	(global_label "V4"
 		(shape input)
@@
 		)
 	)
-	(global_label "RESET"
-		(shape input)
-		(at 81.28 118.11 0)
-		(fields_autoplaced yes)
-		(effects
-			(font
-				(size 1.27 1.27)
-			)
-			(justify left)
-		)
-		(property "Intersheetrefs" "${INTERSHEET_REFS}"
-			(at 90.0103 118.11 0)
-			(effects
-				(font
-					(size 1.27 1.27)
-				)
-				(justify left)
-				(hide yes)
-			)
-		)
-	)
 	(global_label "SPEED3"
 		(shape input)
@@
 		)
 	)
-	(global_label "D-"
-		(shape input)
-		(at 81.28 100.33 0)
-		(fields_autoplaced yes)
-		(effects
-			(font
-				(size 1.27 1.27)
-			)
-			(justify left)
-		)
-		(property "Intersheetrefs" "${INTERSHEET_REFS}"
-			(at 87.1076 100.33 0)
-			(effects
-				(font
-					(size 1.27 1.27)
-				)
-				(justify left)
-				(hide yes)
-			)
-		)
-	)
 	(global_label "U2"
 		(shape input)
@@
 		(fields_autoplaced yes)
 		(property "Reference" "J3"
-			(at 135.89 423.9261 0)
+			(at 139.8972 415.29 0)
 			(effects
 				(font
 					(size 1.27 1.27)
 				)
-				(justify left)
 			)
 		)
 		(property "Value" "U.FL-R-SMT-1_80_"
-			(at 135.89 421.3861 0)
+			(at 139.8972 417.83 0)
 			(effects
 				(font
 					(size 1.27 1.27)
 				)
-				(justify left)
 			)
 		)
@@
 		(fields_autoplaced yes)
 		(property "Reference" "J4"
-			(at 303.53 389.89 90)
+			(at 311.15 350.52 0)
 			(effects
 				(font
@@
 		)
 		(property "Value" "FFC2B28-24-G"
-			(at 300.99 389.89 90)
+			(at 311.15 353.06 0)
 			(effects
 				(font
@@
 		(fields_autoplaced yes)
 		(property "Reference" "D5"
-			(at 170.18 52.07 0)
+			(at 184.15 50.7999 90)
 			(effects
 				(font
 					(size 1.27 1.27)
 				)
+				(justify right)
 			)
 		)
 		(property "Value" "TPD2E001DZDR"
-			(at 172.72 52.07 0)
+			(at 184.15 53.3399 90)
 			(effects
 				(font
 					(size 1.27 1.27)
 				)
+				(justify right)
 			)
 		)
